Commit message: correct urdf for gripper Idol

File: src/bcn3d_description/urdf/moveo.urdf.xacro (robot description, xacro)
@@ -585,10 +585,10 @@
       xyz="0 1 0" />
     <limit
-      lower="-1.5"
-      upper="0"
+      lower="0"
+      upper="1.5"
       effort="10"
       velocity="1" />
       <dynamics damping="0.2" friction="0.02"/>
-      <mimic joint="Gripper_Servo_Gear_Joint" multiplier="-1" offset="0"/>
+      <mimic joint="Gripper_Servo_Gear_Joint" multiplier="1" offset="0"/>
   </joint>
   <link

File: src/bcn3d_gazebo/urdf/moveo_gazebo.urdf.xacro (robot description, xacro)
@@ -126,5 +126,5 @@
       <joint>Gripper_Servo_Gear_Joint</joint>
       <mimicJoint>Tip_Gripper_Idol_Joint</mimicJoint>
-      <multiplier>-1.0</multiplier>
+      <multiplier>1.0</multiplier>
       <offset>0.0</offset>
       <maxEffort>2.0</maxEffort>

Commit message: add realsense d435 in gazebo to visualize the camera frame and the TF

File: src/bcn3d_description/urdf/moveo.urdf.xacro (robot description, xacro)
@@ -745,11 +745,10 @@
        real realsense2_camera driver's TF tree. -->
   <!-- Camera DISABLED for now — realsense xacro bloats URDF past rcl's CLI parser limit.
-       Re-enable when gazebo_ros2_control can handle a larger URDF.
-  <xacro:sensor_d435 parent="Link_5" name="camera" use_nominal_extrinsics="true">
+       Re-enable when gazebo_ros2_control can handle a larger URDF. -->
+  <xacro:sensor_d435 parent="Link_5" name="d435" use_nominal_extrinsics="true" use_mesh="true">
     <origin xyz="-0.04 0 0.06" rpy="0 -0.65 3.1416"/>
   </xacro:sensor_d435>
-  -->
   <!-- Tiny placeholder camera_link so other code that references it still finds the frame -->
-  <link name="camera_link">
+  <!-- <link name="camera_link">
     <inertial>
       <origin xyz="0 0 0" rpy="0 0 0"/>
@@ -762,4 +761,4 @@
     <parent link="Link_5"/>
     <child link="camera_link"/>
-  </joint>
+  </joint> -->
 </robot>

File: src/bcn3d_gazebo/urdf/moveo_gazebo.urdf.xacro (robot description, xacro)
@@ -149,9 +149,34 @@
   </gazebo>
   <!-- Camera sensor temporarily disabled — re-enable with realsense xacro
-       once URDF size is no longer an issue.
-  <gazebo reference="camera_link">
-    <sensor name="camera" type="depth">
+       once URDF size is no longer an issue. -->
+  <gazebo reference="d435_depth_frame">
+    <sensor name="d435_depth" type="depth">
       <update_rate>30</update_rate>
-      <camera name="camera">
+      <visualize>true</visualize>
+      <camera>
+        <horizontal_fov>1.5009</horizontal_fov>
+        <image>
+          <width>848</width>
+          <height>480</height>
+          <format>R_FLOAT32</format>
+        </image>
+        <clip>
+          <near>0.1</near>
+          <far>10.0</far>
+        </clip>
+      </camera>
+      <plugin name="d435_depth_controller" filename="libgazebo_ros_camera.so">
+        <camera_name>d435/depth</camera_name>
+        <frame_name>d435_depth_optical_frame</frame_name>
+        <pointCloudCutoff>0.1</pointCloudCutoff>
+        <pointCloudCutoffMax>5.0</pointCloudCutoffMax>
+      </plugin>
+    </sensor>
+  </gazebo>
+  <gazebo reference="d435_color_frame">
+    <sensor name="d435_color" type="camera">
+      <update_rate>30</update_rate>
+      <visualize>true</visualize>
+      <camera>
         <horizontal_fov>1.5009</horizontal_fov>
         <image>
@@ -165,12 +190,9 @@
         </clip>
       </camera>
-      <plugin name="camera_controller" filename="libgazebo_ros_camera.so">
-        <frame_name>camera_depth_optical_frame</frame_name>
-        <camera_name>camera</camera_name>
-        <pointCloudCutoff>0.1</pointCloudCutoff>
-        <pointCloudCutoffMax>5.0</pointCloudCutoffMax>
+      <plugin name="d435_color_controller" filename="libgazebo_ros_camera.so">
+        <camera_name>d435/color</camera_name>
+        <frame_name>d435_color_optical_frame</frame_name>
       </plugin>
     </sensor>
   </gazebo>
-  -->
 </robot>
